File: esp32-pico-d4-module.kicad_pcb (KiCad board)
At the start: 2 copper layers, 20.6 x 15.6 mm, 11 parts, among them J1 Conn_01x08_Male, J2 Conn_01x08_Male, U1 ESP32_PICO-D4, U2 Trace

Commit message: Documentations, license and improved silk screen
Parts:
- renumbered R2 to R1
Changed lines of the file:
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@@
   (general
     (thickness 1.6)
-    (drawings 40)
-    (tracks 191)
+    (drawings 41)
+    (tracks 190)
     (zones 0)
     (modules 11)
@@
     (tags resistor)
     (attr smd)
-    (fp_text reference R2 (at 0 -1.65) (layer F.SilkS) hide
+    (fp_text reference R1 (at 0 -1.65) (layer F.SilkS) hide
       (effects (font (size 1 1) (thickness 0.15)))
     )
@@
       (net 15 /IO18))
   )
+  (gr_text "Thingler\nESP32\nModule\nV1.0" (at 122.5 109.4) (layer F.SilkS)
+    (effects (font (size 0.7 0.7) (thickness 0.12)) (justify left))
+  )
   (gr_text 22 (at 124.75 113.1) (layer F.SilkS)
     (effects (font (size 0.8 0.8) (thickness 0.12)))
@@
   )
   (segment (start 123.35 106.4125) (end 123.4625 106.3) (width 0.25) (layer F.Cu) (net 2))
-  (segment (start 122.55 106.4125) (end 123.35 106.4125) (width 0.25) (layer F.Cu) (net 2))
+  (segment (start 122.55 106.4125) (end 123.35 106.4125) (width 0.25) (layer F.Cu) (net 2) (status 10))
   (segment (start 123.4625 106.3) (end 123.9 106.3) (width 0.25) (layer F.Cu) (net 2))
   (segment (start 123.9 106.3) (end 123.9 106.1) (width 0.25) (layer F.Cu) (net 2))
@@
   (segment (start 121.32501 106.12499) (end 121.32501 104.77501) (width 0.25) (layer F.Cu) (net 4))
   (segment (start 120.125 104.4) (end 120.95 104.4) (width 0.25) (layer F.Cu) (net 4))
-  (segment (start 119.875 104.65) (end 120.125 104.4) (width 0.25) (layer F.Cu) (net 4))
+  (segment (start 119.875 104.65) (end 120.125 104.4) (width 0.25) (layer F.Cu) (net 4) (status 10))
   (segment (start 120.95 104.4) (end 121 104.45) (width 0.25) (layer F.Cu) (net 4))
   (via (at 121 104.45) (size 0.6) (drill 0.3) (layers F.Cu B.Cu) (net 4))
-  (segment (start 120.8 111.9) (end 120.8 111.9) (width 0.25) (layer F.Cu) (net 4))
   (segment (start 120.8 111.9) (end 120.8 112) (width 0.25) (layer F.Cu) (net 4))
   (via (at 120.8 111.9) (size 0.6) (drill 0.3) (layers F.Cu B.Cu) (net 4))
@@
   (segment (start 118.5875 103.7875) (end 119.22499 104.42499) (width 0.25) (layer B.Cu) (net 4))
   (segment (start 120.575 111.675) (end 120.8 111.9) (width 0.25) (layer F.Cu) (net 4))
-  (segment (start 120.575 110.85) (end 120.575 111.675) (width 0.25) (layer F.Cu) (net 4))
+  (segment (start 120.575 110.85) (end 120.575 111.675) (width 0.25) (layer F.Cu) (net 4) (status 10))
   (segment (start 122.55 103.625) (end 122.55 103.575) (width 0.25) (layer F.Cu) (net 5))
   (segment (start 122.55 103.725) (end 122.55 103.625) (width 0.25) (layer F.Cu) (net 5))
@@
   (segment (start 124.275 112.55) (end 123.975 112.25) (width 0.25) (layer F.Cu) (net 5))
   (segment (start 126.2875 112.55) (end 124.275 112.55) (width 0.25) (layer F.Cu) (net 5) (status 10))
-  (segment (start 119.375 103.925) (end 119.375 104.65) (width 0.25) (layer F.Cu) (net 5))
+  (segment (start 119.375 103.925) (end 119.375 104.65) (width 0.25) (layer F.Cu) (net 5) (status 20))
   (segment (start 119.675 103.625) (end 119.375 103.925) (width 0.25) (layer F.Cu) (net 5))
   (segment (start 122.55 103.625) (end 119.675 103.625) (width 0.25) (layer F.Cu) (net 5))
@@
   (segment (start 109.75 112.825) (end 109.42501 112.50001) (width 0.25) (layer B.Cu) (net 6))
   (segment (start 115.875 103.75) (end 115.92499 103.70001) (width 0.25) (layer F.Cu) (net 6))
-  (segment (start 115.875 104.65) (end 115.875 103.75) (width 0.25) (layer F.Cu) (net 6))
+  (segment (start 115.875 104.65) (end 115.875 103.75) (width 0.25) (layer F.Cu) (net 6) (status 10))
   (via (at 113.475 112.8) (size 0.6) (drill 0.3) (layers F.Cu B.Cu) (net 7))
   (segment (start 112.1 111.6) (end 113.3 112.8) (width 0.25) (layer F.Cu) (net 7))
@@
   (segment (start 113.675 109.35) (end 112.65 109.35) (width 0.25) (layer F.Cu) (net 7) (status 10))
   (segment (start 121.8 103.3) (end 122.124999 102.975001) (width 0.25) (layer B.Cu) (net 7))
-  (segment (start 126.730001 102.649999) (end 127.58 101.8) (width 0.25) (layer B.Cu) (net 7))
+  (segment (start 126.730001 102.649999) (end 127.58 101.8) (width 0.25) (layer B.Cu) (net 7) (status 20))
   (segment (start 126.404999 102.975001) (end 126.730001 102.649999) (width 0.25) (layer B.Cu) (net 7))
   (segment (start 123.200011 106.075011) (end 121.8 104.675) (width 0.25) (layer B.Cu) (net 7))
@@
   (segment (start 123.849991 113.299991) (end 122.750001 112.200001) (width 0.25) (layer F.Cu) (net 11))
   (segment (start 122.750001 112.200001) (end 122.750001 108.324999) (width 0.25) (layer F.Cu) (net 11))
-  (segment (start 124.190001 113.750001) (end 125.04 114.6) (width 0.25) (layer F.Cu) (net 12))
+  (segment (start 124.190001 113.750001) (end 125.04 114.6) (width 0.25) (layer F.Cu) (net 12) (status 20))
   (segment (start 123.600001 113.750001) (end 124.190001 113.750001) (width 0.25) (layer F.Cu) (net 12))
   (segment (start 122.2 110.63859) (end 122.2 112.35) (width 0.25) (layer F.Cu) (net 12))
   (segment (start 121.41141 109.85) (end 122.2 110.63859) (width 0.25) (layer F.Cu) (net 12))
   (segment (start 122.2 112.35) (end 123.600001 113.750001) (width 0.25) (layer F.Cu) (net 12))
-  (segment (start 120.575 109.85) (end 121.41141 109.85) (width 0.25) (layer F.Cu) (net 12))
+  (segment (start 120.575 109.85) (end 121.41141 109.85) (width 0.25) (layer F.Cu) (net 12) (status 10))
   (segment (start 119.875 114.515) (end 119.96 114.6) (width 0.25) (layer F.Cu) (net 13) (status 30))
   (segment (start 119.875 111.55) (end 119.875 114.515) (width 0.25) (layer F.Cu) (net 13) (status 30))
